File: bob/bob.kicad_sch (KiCad schematic)
At the start: 0 parts

Commit message: WIP
Parts:
- added U1: PY32F071R1xU6, Package_DFN_QFN:QFN-64-1EP_8x8mm_P0.4mm_EP6.5x6.5mm, symbol MCU_Puya_PY32F:PY32F071R1xU6
- added X1: SWD, drake:SWD, symbol Drake:SWD

Commit message: WIP
Parts:
- removed U1: PY32F071R1xU6, Package_DFN_QFN:QFN-64-1EP_8x8mm_P0.4mm_EP6.5x6.5mm, symbol MCU_Puya_PY32F:PY32F071R1xU6
- removed X1: SWD, drake:SWD, symbol Drake:SWD
- added A1: 31mm, Connector_Wire:SolderWire-1.5sqmm_1x01_D1.7mm_OD3.9mm, symbol Device:Antenna
- added C1, C2, C3, C4: NC, Capacitor_SMD:C_0805_2012Metric, symbol Device:C
- added C10, C12, C6, C9: 100n, Capacitor_SMD:C_0805_2012Metric, symbol Device:C
- added C11, C7: 10u, Capacitor_SMD:C_0805_2012Metric, symbol Device:C
- added C5, C8: 1u, Capacitor_SMD:C_0805_2012Metric, symbol Device:C
- added D1: RED, LED_SMD:LED_0805_2012Metric, symbol Device:LED
- added D2: GREEN, LED_SMD:LED_0805_2012Metric, symbol Device:LED
- added J1: PROG, Connector_PinHeader_2.54mm:PinHeader_2x05_P2.54mm_Vertical, symbol Connector_Generic:Conn_02x05_Odd_Even
- added J2: PHL, Connector_PinHeader_2.54mm:PinHeader_1x11_P2.54mm_Vertical, symbol Connector:Conn_01x12_Pin
- added J3: PHR, Connector_PinHeader_2.54mm:PinHeader_1x11_P2.54mm_Vertical, symbol Connector:Conn_01x12_Pin
- added R1: 0R, Resistor_SMD:R_0805_2012Metric, symbol Device:R
- added R3, R4: 270R, Resistor_SMD:R_0805_2012Metric, symbol Device:R
- added U1: PAN2110P0AA, Package_SO:SOIC-8_3.9x4.9mm_P1.27mm, symbol Drake:PAN2110P0AA
- added U2: LM1117MP-3.3, Package_TO_SOT_SMD:SOT-223-3_TabPin2, symbol Regulator_Linear:LM1117MP-3.3
- added U3: PY32F030K1xTx, Package_QFP:LQFP-32_7x7mm_P0.8mm, symbol MCU_Puya_PY32F:PY32F030K1xTx
- added Y1: 16MHz, Crystal:Crystal_SMD_3225-4Pin_3.2x2.5mm, symbol Device:Crystal_GND24_Small
Connections:
- new net: D1.2 (A), R3.2
- new net: C4.2, U1.5 (XC1), Y1.1
- new net: C3.2, U1.6 (XC0), Y1.3
- new net: C2.2, R1.1, U1.8 (ANT)
- new net: A1.1 (A), C1.2, R1.2
- new net: D2.2 (A), R4.2
- new net: C9.1, U3.4 (PF2-NRST)
- new net +3V3: C10.1, C11.1, C12.1, C5.1, C6.1, C8.1, J1.1 (Pin_1), J1.2 (Pin_2), J2.3 (Pin_3), U1.4 (VDD), U2.2 (VO), U3.1 (VCC), U3.17 (VCC)
- new net +5V: C7.1, J1.10 (Pin_10), J1.9 (Pin_9), J2.2 (Pin_2), U2.3 (VI)
- new net GND: C1.1, C10.2, C11.2, C12.2, C2.1, C3.1, C4.1, C5.2, C6.2, C7.2, C8.2, C9.2, D1.1 (K), D2.1 (K), J1.7 (Pin_7), J1.8 (Pin_8), J2.1 (Pin_1), J3.1 (Pin_1), U1.7 (VSS), U2.1 (GND), U3.16 (VSS), U3.32 (VSS), Y1.2 (G), Y1.4 (G)
- new net PA0: J3.2 (Pin_2), U3.6 (PA0)
- new net PA1: J3.3 (Pin_3), U3.7 (PA1)
- new net PA11: J3.10 (Pin_10), U3.21 (PA11)
- new net PA12: J3.11 (Pin_11), U3.22 (PA12)
- new net PA15: J3.12 (Pin_12), U3.25 (PA15)
- new net PA2: J3.4 (Pin_4), U3.8 (PA2)
- new net PA3: J3.5 (Pin_5), U3.9 (PA3)
- new net PA4: J3.6 (Pin_6), U3.10 (PA4)
- new net PA5: J3.7 (Pin_7), U3.11 (PA5)
- new net PA6: J3.8 (Pin_8), U3.12 (PA6)
- new net PA8: J3.9 (Pin_9), U3.18 (PA8)
- new net PB0: J2.8 (Pin_8), R3.1, U3.14 (PB0)
- new net PB1: J2.9 (Pin_9), R4.1, U3.15 (PB1)
- new net PB3: J2.10 (Pin_10), U3.26 (PB3)
- new net PB4: J2.11 (Pin_11), U3.27 (PB4)
- new net PB5: J2.12 (Pin_12), U3.28 (PB5)
- new net PF0: J2.4 (Pin_4), U3.2 (PF0-OSCIN)
- new net PF1: J2.5 (Pin_5), U3.3 (PF1-OSCOUT)
- new net PF3: J2.6 (Pin_6), U3.5 (PF3)
- new net PF4: J2.7 (Pin_7), U3.31 (PF4-BT0)
- new net PROG_CLK: J1.6 (Pin_6), U3.24 (PA14-SWC)
- new net PROG_DIO: J1.4 (Pin_4), U3.23 (PA13-SWD)
- new net PROG_RXD: J1.5 (Pin_5), U3.30 (PB7)
- new net PROG_TXD: J1.3 (Pin_3), U3.29 (PB6)
- new net RF_CLK: U1.2 (SCL/SCK), U3.19 (PA9-OSC32OUT)
- new net RF_DIO: U1.3 (SDA/DATA), U3.13 (PA7)
- new net ~{RF_CS}: U1.1 (CSN), U3.20 (PA10-OSC32IN)
Other:
- note added: "PA7: SPI1_MOSI / I2C_SDA PA9: SPI1_SCK / I2C_SCL PA10: SPI1_NSS"

Commit message: WIP
Parts:
- added D1: DSK14, Diode_SMD:D_SOD-123, symbol Device:D
- added JP1: 5V / 3.3V, Jumper:SolderJumper-3_P2.0mm_Open_TrianglePad1.0x1.5mm, symbol Jumper:SolderJumper_3_Open
- added R2: 0R, Resistor_SMD:R_0805_2012Metric, symbol Device:R
- A1: footprint Connector_Wire:SolderWire-1.5sqmm_1x01_D1.7mm_OD3.9mm -> Drake:Wire antena 2.4GHz
- J2: renamed from J3; value PHR -> PWR; footprint Connector_PinHeader_2.54mm:PinHeader_1x11_P2.54mm_Vertical -> Connector_PinHeader_2.54mm:PinHeader_1x02_P2.54mm_Vertical; symbol Connector:Conn_01x12_Pin -> Connector:Conn_01x02_Pin
- J3: renamed from J2; value PHL -> BB; footprint Connector_PinHeader_2.54mm:PinHeader_1x11_P2.54mm_Vertical -> Connector_PinHeader_2.54mm:PinHeader_1x24_P2.54mm_Vertical; symbol Connector:Conn_01x12_Pin -> Connector:Conn_01x24_Pin
- renumbered C9 to C10, C8 to C7, C10 to C8, C7 to C9, D1 to D2, D2 to D3
Connections:
- net +3V3: now also D1.1 (K), JP1.1 (A); no longer C11.1, U2.2 (VO)
- net +5V: now also JP1.3 (B)
- net GND: now also J3.24 (Pin_24)
- net PA0: now also J3.4 (Pin_4); no longer J2.2 (Pin_2)
- net PA1: now also J3.5 (Pin_5); no longer J2.3 (Pin_3)
- net PA11: now also J3.12 (Pin_12); no longer J2.10 (Pin_10)
- net PA12: now also J3.13 (Pin_13); no longer J2.11 (Pin_11)
- net PA15: now also J3.14 (Pin_14); no longer J2.12 (Pin_12)
- net PA2: now also J3.6 (Pin_6); no longer J2.4 (Pin_4)
- net PA3: now also J3.7 (Pin_7); no longer J2.5 (Pin_5)
- net PA4: now also J3.8 (Pin_8); no longer J2.6 (Pin_6)
- net PA5: now also J3.9 (Pin_9); no longer J2.7 (Pin_7)
- net PA6: now also J3.10 (Pin_10); no longer J2.8 (Pin_8)
- net PA8: now also J3.11 (Pin_11); no longer J2.9 (Pin_9)
- net PB0: now also J3.19 (Pin_19); no longer J3.8 (Pin_8)
- net PB1: now also J3.20 (Pin_20); no longer J3.9 (Pin_9)
- net PB3: now also J3.21 (Pin_21); no longer J3.10 (Pin_10)
- net PB4: now also J3.22 (Pin_22); no longer J3.11 (Pin_11)
- net PB5: now also J3.23 (Pin_23); no longer J3.12 (Pin_12)
- net PF0: now also J3.15 (Pin_15); no longer J3.4 (Pin_4)
- net PF1: now also J3.16 (Pin_16); no longer J3.5 (Pin_5)
- net PF3: now also J3.17 (Pin_17); no longer J3.6 (Pin_6)
- net PF4: now also J3.18 (Pin_18); no longer J3.7 (Pin_7)
- net at C4.2, Y1.1: now also R2.2; no longer U1.5 (XC1)
- new net: C11.1, D1.2 (A), U2.2 (VO)
- new net: R2.1, U1.5 (XC1)
- new net: J2.2 (Pin_2), JP1.2 (C)
Other:
- moved on the sheet: A1, C1, C2, C3, C4, R1, Y1
