File: bob/bob.kicad_pcb (KiCad board)
At the start: 2 copper layers, 25 parts, among them J1 PROG, J2 PHL, J3 PHR, U1 PAN2110P0AA, U2 LM1117MP-3.3, U3 PY32F030K1xTx, Y1 16MHz

Commit message: WIP
Parts:
- added D1: DSK14, Diode_SMD:D_SOD-123, F.Cu at (204.0, 53.0)
- added JP1: 5V / 3.3V, Jumper:SolderJumper-3_P2.0mm_Open_TrianglePad1.0x1.5mm, F.Cu at (182.0, 54.5)
- added R2: 0R, Resistor_SMD:R_0805_2012Metric, F.Cu at (235.5, 64.0)
- A1: footprint Connector_Wire:SolderWire-1.5sqmm_1x01_D1.7mm_OD3.9mm -> Drake:Wire antena 2.4GHz
- J2: renamed from J3; value PHR -> PWR; footprint Connector_PinHeader_2.54mm:PinHeader_1x11_P2.54mm_Vertical -> Connector_PinHeader_2.54mm:PinHeader_1x02_P2.54mm_Vertical
- J3: renamed from J2; value PHL -> BB; footprint Connector_PinHeader_2.54mm:PinHeader_1x11_P2.54mm_Vertical -> Connector_PinHeader_2.54mm:PinHeader_1x24_P2.54mm_Vertical
- moved U1 89.7 mm to (233.0, 60.0), turned to 0 degrees
- moved U2 62.1 mm to (199.0, 59.0), turned to -90 degrees
- moved D2 51.9 mm to (205.0, 57.0), turned to -90 degrees
- moved D3 51.3 mm to (205.0, 61.0), turned to -90 degrees
- moved R3 43.9 mm to (207.5, 57.0), turned to 90 degrees
- moved R4 43.5 mm to (207.5, 61.0), turned to -90 degrees
- moved U3 39.3 mm to (216.5, 59.1), turned to -90 degrees
- moved A1 37.3 mm to (239.5, 53.0), turned to 90 degrees
- moved C12 31.3 mm to (206.5, 64.0), turned to 180 degrees
- moved C9 25.3 mm to (195.5, 53.0), turned to 0 degrees
- moved R1 23.3 mm to (235.5, 53.5), turned to 90 degrees
- moved C11 20.2 mm to (199.5, 53.0), turned to 180 degrees
- moved C8 18.1 mm to (223.0, 53.5), turned to 90 degrees
- moved C7 18.1 mm to (228.0, 53.5), turned to 90 degrees
- moved C3 15.2 mm to (239.5, 58.0)
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- renumbered C9 to C10, C8 to C7, C10 to C8, C7 to C9, D1 to D2, D2 to D3
Connections:
- C11 pad 1: +3V3 -> Net-(D1-A)
- C4 pad 2: Net-(U1-XC1) -> Net-(C4-Pad2)
- J2 pad 2: /PA0 -> Net-(J2-Pin_2)
- J3 pad 10: /PB3 -> /PA6
- J3 pad 11: /PB4 -> /PA8
- J3 pad 4: /PF0 -> /PA0
- J3 pad 5: /PF1 -> /PA1
- J3 pad 6: /PF3 -> /PA2
- J3 pad 7: /PF4 -> /PA3
- J3 pad 8: /PB0 -> /PA4
- J3 pad 9: /PB1 -> /PA5
- U2 pad 2: +3V3 -> Net-(D1-A)
- Y1 pad 1: Net-(U1-XC1) -> Net-(C4-Pad2)
Routing:
- net /PA0: track 0.00 -> 37.8 mm, vias 0 -> 1
- net /PROG_CLK: track 0.00 -> 37.1 mm, vias 0 -> 2
- net /PROG_DIO: track 0.00 -> 36.2 mm, vias 0 -> 2
- net /PA1: track 0.00 -> 35.3 mm, vias 0 -> 1
- net GND: track 0.00 -> 35.2 mm, vias 0 -> 19
- net /PB1: track 0.00 -> 35.0 mm, vias 0 -> 3
- net /PROG_TXD: track 0.00 -> 33.4 mm, vias 0 -> 2
- net /PA2: track 0.00 -> 32.5 mm, vias 0 -> 1
- net /PROG_RXD: track 0.00 -> 32.4 mm, vias 0 -> 2
- net +5V: track 0.00 -> 32.2 mm
- net /PB0: track 0.00 -> 31.1 mm, vias 0 -> 2
- net /RF_DIO: track 0.00 -> 26.7 mm, vias 0 -> 2
- net /PF3: track 0.00 -> 26.3 mm, vias 0 -> 2
- net /PF1: track 0.00 -> 26.0 mm, vias 0 -> 4
- net +3V3: track 0.00 -> 25.0 mm, vias 0 -> 7
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- added copper zone on In2.Cu, net +3V3
- added copper zone on In1.Cu, net GND
Other:
- board outline added: 62 x 19 mm
- copper layers 2 -> 4
- board text added: "${REFERENCE}"
- board text added: "3V3"
- board text added: "5V"
- board text added: "A0"
- board text added: "A1"
- board text added: "A11"
- board text added: "A12"
- board text added: "A15"
- board text added: "A2"
- board text added: "A3"
- board text added: "A4"
- board text added: "A5"
- board text added: "A6"
- board text added: "A8"
- board text added: "B0"
- board text added: "B1"
- board text added: "B3"
- board text added: "B4"
- board text added: "B5"
- board text added: "BLÉ-RIOT"
- board text added: "BOB v1.0"
- board text added: "BT"
- board text added: "F0"
- board text added: "F1"
- board text added: "F3"
- board text added: "F4"
- board text added: "GND"
- board text added: "LG"
- board text added: "LR"
- board text added: "RX"
- board text added: "SWC"
- board text added: "SWD"
- board text added: "TX"

Commit message: WIP
Parts:
- moved C2 3.48 mm to (233.8, 54.8), turned to 0 degrees
- moved R1 2.50 mm to (237.5, 55.0), turned to 45 degrees
- moved C1 1.25 mm to (233.8, 52.5), turned to 0 degrees
Routing:
- net Net-(U1-ANT): track 9.31 -> 0.00 mm
- net Net-(A1-A): track 6.69 -> 0.00 mm
- net GND: track 35.2 -> 32.1 mm, vias 19 -> 18
Other:
- board text added: "BOB v1.1"
- board text added: "Doladit anténu - zkrátit připojení kondenzátorů. Navrhnout správně Microstrip nebo Grounded coplanar waveguide."
- board text removed: "BOB v1.0"
